Commit message: camera done

File: src/dobot_gazebo/urdf/camera.xacro (robot description, xacro)
@@ -19,5 +19,5 @@
             </visual>
             <collision>
-                <origin xyz="0.0 0.0 0.0" rpy="0 0 0" />
+                <origin xyz="0.0 0.0 0.0" rpy="0 1.57 0" />
                 <geometry>
                     <box size="0.01 0.04 0.04" />

File: src/dobot_gazebo/urdf/cr5_robot_camera.xacro (robot description, xacro)
@@ -3,11 +3,11 @@
     <xacro:include filename="$(find dobot_gazebo)/urdf/cr5_robot.xacro"/>
     <xacro:include filename="$(find dobot_gazebo)/urdf/camera.xacro"/>
-    <xacro:property name="camera_offset_x" value="0.3" />
-    <xacro:property name="camera_offset_y" value="0" />
-    <xacro:property name="camera_offset_z" value="0.14" />
+    <xacro:property name="camera_offset_x" value="0" />
+    <xacro:property name="camera_offset_y" value="-0.5" />
+    <xacro:property name="camera_offset_z" value="2.5" />
     <robot_base/>
     <!-- Camera -->
     <joint name="camera_joint" type="fixed">
-        <origin xyz="${camera_offset_x} ${camera_offset_y} ${camera_offset_z}" rpy="0 0 0" />
+        <origin xyz="${camera_offset_x} ${camera_offset_y} ${camera_offset_z}" rpy="0 1.5707 0" />
         <parent link="base_link"/>
         <child link="camera_link"/>

Commit message: get picture but the tag mismatch

File: src/dobot_gazebo/urdf/camera.xacro (robot description, xacro)
@@ -19,5 +19,5 @@
             </visual>
             <collision>
-                <origin xyz="0.0 0.0 0.0" rpy="0 1.57 0" />
+                <origin xyz="0.0 0.0 0.0" rpy="0 0 0" />
                 <geometry>
                     <box size="0.01 0.04 0.04" />

Commit message: change camera angel, picture and position differ by one frame

File: src/dobot_gazebo/urdf/camera.xacro (robot description, xacro)
@@ -34,5 +34,5 @@
                     <horizontal_fov>1.3962634</horizontal_fov>
                     <image>
-                        <width>1280</width>
+                        <width>1000</width>
                         <height>720</height>
                         <format>R8G8B8</format>

File: src/dobot_gazebo/urdf/cr5_robot_camera.xacro (robot description, xacro)
@@ -4,10 +4,10 @@
     <xacro:include filename="$(find dobot_gazebo)/urdf/camera.xacro"/>
     <xacro:property name="camera_offset_x" value="0" />
-    <xacro:property name="camera_offset_y" value="-0.5" />
-    <xacro:property name="camera_offset_z" value="2.5" />
+    <xacro:property name="camera_offset_y" value="-0.7" />
+    <xacro:property name="camera_offset_z" value="1.8" />
     <robot_base/>
     <!-- Camera -->
     <joint name="camera_joint" type="fixed">
-        <origin xyz="${camera_offset_x} ${camera_offset_y} ${camera_offset_z}" rpy="0 1.5707 0" />
+        <origin xyz="${camera_offset_x} ${camera_offset_y} ${camera_offset_z}" rpy="-1.5707963 1.5707963 0" />
         <parent link="base_link"/>
         <child link="camera_link"/>
